File: fram80.kicad_sch (KiCad schematic)
At the start: 12 parts, among them J1 UPPER, J2 LOWER, U1 FM1808B-SG, U3 74LS00

Commit message: Support upper 32K
Parts:
- added JP4: UPPER, Connector_PinHeader_2.54mm:PinHeader_1x03_P2.54mm_Vertical, symbol Jumper:Jumper_3_Open
- added U4: 74HCT00, Package_SO:TSSOP-14_4.4x5mm_P0.65mm, symbol 74xx:74LS00
- U3: value 74LS00 -> 74HCT00; footprint Package_SO:SO-14_3.9x8.65mm_P1.27mm -> Package_SO:TSSOP-14_4.4x5mm_P0.65mm
Connections:
- net +5V: now also U4.10, U4.14 (VCC), U4.9
- net A10: now also U3.4, U3.5; no longer U3.1, U3.2
- net GND: now also U4.7 (GND)
- net ~{A10}: now also U3.6; no longer U3.3
- net ~{CS}: now also U4.6; no longer U3.8
- net ~{MEMR}: now also U3.2; no longer U3.5
- net ~{MEMW}: now also U3.1; no longer U3.4
- net ~{SEL0}: now also U4.12, U4.13; no longer U3.12, U3.13
- net at U3.11: now also U4.4; no longer U3.10
- net A15: now reaches J1.20 (Pin_20)
- net A15: now also U3.10, U3.9, JP4.1 (A)
- new net: U4.1, U4.11
- new net: JP4.2 (C), U4.2
- new net: U3.12, U3.13, U4.3
- new net: U3.3, U4.5
- new net ~{A15}: JP4.3 (B), U3.8
- no-connect marks 1 -> 2
Other:
- note added: "~{CS} = (~{MEMW} OR ~{MEMR}) AND ~{SEL0} AND A15"
- moved on the sheet: C1, JP2, R1, U3B, U3C, U3D
